File: PCB/MSI LED Driver/Initial Design.sch (KiCad schematic (older format))
At the start: 30 parts, among them J1 , J2 , J3 RJ45, J4 , J5 , J6 , Q1 , U1 , U10 , U11 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

Commit message: Fix
Other:
- note added: "Does this need a\npull-down resistor?"
- note removed: "Does this need a\npull-up resistor?"
Changed lines of the file:
@@
 Wire Wire Line
 	4975 5400 5025 5400
-Text Notes 4900 5750 0    50   ~ 0
-Does this need a\npull-up resistor?
+Text Notes 4850 5700 0    50   ~ 0
+Does this need a\npull-down resistor?
 Text GLabel 5750 4750 2    50   Input ~ 0
 C2
